Commit message: for tracking

File: data/dummy_urdf/dummy.urdf (robot description, URDF)
Before this commit: robot dummy, 9 links, 8 joints
Links:
- link tool0: geometry collision box size=0.04 0.04 0.1; visual box size=0.04 0.04 0.1

Commit message: update j6

File: data/dummy_urdf/dummy.urdf (robot description, URDF)
Before this commit: robot dummy, 9 links, 8 joints
Joints:
- joint Joint6: limit lower=-3.14 upper=3.14 effort=150 velocity=3.15 -> lower=-3.14 upper=3.14 effort=150 velocity=1.00
